Commit message: feat: 作业3.2 - src-1

File: 人形机器人综合实践课(2025年1期)/三、机器人建模与可视化/作业3.2/src/arm_5dof/urdf/arm_5dof.urdf (robot description, URDF)
Before this commit: robot arm_5dof, 6 links, 5 joints
Joints:
- joint joint_1: origin xyz=0 0 0.05 rpy=1.5708 0 0 -> xyz=0 0 0.05 rpy=0 0 0
- joint joint_3: limit lower=-1 upper=1 effort=10 velocity=1 -> lower=-2 upper=2 effort=10 velocity=1
