Commit message: fix: 作业3.2 - complete

File: 人形机器人综合实践课(2025年1期)/三、机器人建模与可视化/作业3.2/src/arm_5dof/urdf/arm_5dof.urdf (robot description, URDF)
Before this commit: robot arm_5dof, 6 links, 5 joints
Links:
- link base_link: mass 3.61911473693544 -> 10.4022
- link link_1: mass 0.678584013175395 -> 3.29071
- link link_2: mass 1.44 -> 6.22282
- link link_3: mass 0.962112750161874 -> 4.6642
- link link_4: mass 0.339292006587698 -> 1.3415
- link link_5: mass 0.192 -> 0.45494
Joints:
- removed joint joint_1
- removed joint joint_2
- removed joint joint_3
- removed joint joint_4
- removed joint joint_5
- added joint base_yaw: type revolute, parent base_link, child link_1, origin xyz=0 0 0.08 rpy=0 0 0, axis 0 0 1, limit lower=-3.1416 upper=3.1416 effort=30 velocity=1.5
- added joint elbow_pitch: type revolute, parent link_2, child link_3, origin xyz=0 0 0.3 rpy=0 0 0, axis 0 1 0, limit lower=-2.3562 upper=2.3562 effort=20 velocity=1.5
- added joint shoulder_pitch: type revolute, parent link_1, child link_2, origin xyz=0 0 0.06 rpy=0 0 0, axis 0 1 0, limit lower=-1.5708 upper=1.5708 effort=30 velocity=1.5
- added joint wrist_pitch: type revolute, parent link_3, child link_4, origin xyz=0 0 0.37 rpy=0 0 0, axis 0 1 0, limit lower=-2.0944 upper=2.0944 effort=10 velocity=2.0
- added joint wrist_roll: type revolute, parent link_4, child link_5, origin xyz=0 0 0 rpy=0 0 0, axis 0 0 1, limit lower=-3.1416 upper=3.1416 effort=8 velocity=2.5
